File: hardware/harvester_hat.sch (EAGLE design)
At the start: 11 parts, among them IC1 7805T, J1 DCJ0202, U1 CAT24C32

Commit message: added extra files
Parts:
- removed RPI1: RASPBERRYPI_BPLUS_HATNOSLOTS, microbuilder:RASPBERRYPI_BPLUS_HATNOSLOTS
- added AMP: (no value), SparkFun-Connectors:CONN_07
- added J3: RASPBERRYPI-40-PIN-GPIO_PTH, SparkFun-Connectors:RASPBERRYPI-40-PIN-GPIO_PTH
- added S1, S10, S2, S3, S4, S5, S6, S7, S8, S9: MOMENTARY-SWITCH-SPST-PTH-6.0MM, SparkFun-Switches:MOMENTARY-SWITCH-SPST-PTH-6.0MM
- renumbered JP1 to MIC1, JP2 to MIC2
Connections:
- new net N$7: AMP.5
- new net N$8: AMP.4
- net 3.3V: now also J3.3.3V@1, J3.3.3V@17; no longer RPI1.3.3V, RPI1.3.3V@1
- net 5.0V: now also AMP.7, J3.5V@2, J3.5V@4; no longer RPI1.5.0V, RPI1.5.0V@1
- net EECLK: now also J3.ID_SC; no longer RPI1.EECLK
- net EEDATA: now also J3.ID_SD; no longer RPI1.EEDATA
- net GND: now also AMP.6, J3.GND@14, J3.GND@20, J3.GND@25, J3.GND@30, J3.GND@34, J3.GND@39, J3.GND@6, J3.GND@9, S1.2, S10.2, S2.2, S3.2, S4.2, S5.2, S6.2, S7.2, S8.2, S9.2; no longer RPI1.GND, RPI1.GND@1, RPI1.GND@2, RPI1.GND@3, RPI1.GND@4, RPI1.GND@5, RPI1.GND@6, RPI1.GND@7
- net GPIO12: now also J3.GP12, S4.1; no longer RPI1.GPIO12
- net GPIO13: now also J3.GP13, S5.1; no longer RPI1.GPIO13
- net GPIO16: now also J3.GP16, S6.1; no longer RPI1.GPIO16
- net GPIO17: now also J3.GP17, S7.1; no longer RPI1.GPIO17
- net GPIO18: now also AMP.2, J3.GP18#; no longer RPI1.GPIO18
- net GPIO19: now also AMP.1, J3.GP19; no longer RPI1.GPIO19
- net GPIO20: now also J3.GP20; no longer RPI1.GPIO20
- net GPIO21: now also AMP.3, J3.GP21; no longer RPI1.GPIO21
- net GPIO22: now also J3.GP22, S8.1; no longer RPI1.GPIO22
- net GPIO23: now also J3.GP23, S9.1; no longer RPI1.GPIO23
- net GPIO24: now also J3.GP24, S10.1; no longer RPI1.GPIO24
- net GPIO25: now also J3.GP25; no longer RPI1.GPIO25
- net GPIO26: now also J3.GP26; no longer RPI1.GPIO26
- net GPIO27: now also J3.GP27; no longer RPI1.GPIO27
- net GPIO4: now also J3.GP4, S1.1; no longer RPI1.GPIO4
- net GPIO5: now also J3.GP5, S2.1; no longer RPI1.GPIO5
- net GPIO6: now also J3.GP6, S3.1; no longer RPI1.GPIO6
- net RXD: now also J3.RXI; no longer RPI1.RXD
- net SCL: now also J3.SCL; no longer RPI1.SCL
- net SDA: now also J3.SDA; no longer RPI1.SDA
- net SPI_CE0: now also J3.CE0; no longer RPI1.#SPI_CE0
- net SPI_CE1: now also J3.CE1; no longer RPI1.#SPI_CE1
- net SPI_MISO: now also J3.MISO; no longer RPI1.SPI_MISO
- net SPI_MOSI: now also J3.MOSI; no longer RPI1.SPI_MOSI
- net SPI_SCLK: now also J3.SCLK; no longer RPI1.SPI_SCLK
- net TXD: now also J3.TXO; no longer RPI1.TXD
